File: hardware/interface/interface.kicad_pcb (KiCad board)
At the start: 2 copper layers, 63.5 x 22.2 mm, 15 parts, among them J1 Conn_01x04, J2 Conn_01x06, J8 CONN_01X02, Q1 BC547

Commit message: Update.
Parts:
- removed REF** (x4): MountingHole_2.5mm, MountingHole:MountingHole_2.5mm
- added H1: MountingHole, MountingHole:MountingHole_2.7mm_M2.5, F.Cu at (121.3, 73.7)
- added H2: MountingHole, MountingHole:MountingHole_2.7mm_M2.5, F.Cu at (121.3, 88.9)
- added H3: MountingHole, MountingHole:MountingHole_2.7mm_M2.5, F.Cu at (178.4, 73.7)
- added H4: MountingHole, MountingHole:MountingHole_2.7mm_M2.5, F.Cu at (178.4, 88.9)
- added R5: 1K, Resistor_THT:R_Axial_DIN0309_L9.0mm_D3.2mm_P5.08mm_Vertical, F.Cu at (153.7, 80.6)
- J1: value Conn_01x04 -> Switches
- J2: value Conn_01x06 -> Arduino; footprint Connector_PinHeader_2.54mm:PinHeader_1x06_P2.54mm_Vertical -> Connector_PinHeader_2.54mm:PinHeader_1x04_P2.54mm_Vertical
- Q1: footprint Package_TO_SOT_THT:TO-92 -> Package_TO_SOT_THT:TO-92_Wide
- R1: value R -> 1K; footprint Resistor_THT:R_Axial_DIN0309_L9.0mm_D3.2mm_P2.54mm_Vertical -> Resistor_THT:R_Axial_DIN0309_L9.0mm_D3.2mm_P5.08mm_Vertical
- R2: value R -> 2K; footprint Resistor_THT:R_Axial_DIN0309_L9.0mm_D3.2mm_P2.54mm_Vertical -> Resistor_THT:R_Axial_DIN0309_L9.0mm_D3.2mm_P5.08mm_Vertical
- R3: value R -> 4K7; footprint Resistor_THT:R_Axial_DIN0309_L9.0mm_D3.2mm_P2.54mm_Vertical -> Resistor_THT:R_Axial_DIN0309_L9.0mm_D3.2mm_P5.08mm_Vertical
- moved J2 17.0 mm to (157.5, 88.9), turned to 90 degrees
- moved R1 5.46 mm to (161.9, 75.6)
- moved R2 5.46 mm to (161.9, 79.4)
- moved R3 5.46 mm to (161.9, 83.2)
- moved R4 4.58 mm to (154.3, 72.4)
- moved D1 2.84 mm to (151.1, 74.9), turned to 270 degrees
- moved Q1 1.80 mm to (150.5, 83.8)
- moved J1 0.64 mm to (171.4, 85.7)
Connections:
- J2 pad 3: Net-(J1-Pad4) -> Net-(J2-Pad3)
- J2 pad 4: Net-(J1-Pad3) -> GND
- R1 pad 1: Net-(C2-Pad1) -> Net-(J2-Pad3)
- R2 pad 1: Net-(C2-Pad1) -> Net-(J2-Pad3)
- R3 pad 1: Net-(C2-Pad1) -> Net-(J2-Pad3)
- R4 pad 1: Net-(Q1-Pad2) -> Net-(C2-Pad1)
- R4 pad 2: Net-(J2-Pad2) -> Net-(J2-Pad3)
- RLY1 pad 1: Net-(C2-Pad1) -> Net-(D1-Pad1)
- RLY1 pad 16: Net-(D1-Pad1) -> Net-(C2-Pad1)
- RLY1 pad 5: Net-(J8-Pad2) -> Net-(J8-Pad1)
- RLY1 pad 8: Net-(J8-Pad1) -> Net-(J8-Pad2)
Routing:
- net Net-(D1-Pad1): track 12.9 -> 49.4 mm
- net Net-(J2-Pad3): track 0.00 -> 17.8 mm
- net Net-(C2-Pad1): track 57.0 -> 41.1 mm
- net Net-(J1-Pad2): track 11.8 -> 4.46 mm
- net Net-(J1-Pad3): track 11.2 -> 5.00 mm
- net Net-(J2-Pad2): track 3.17 -> 8.78 mm
- net Net-(J1-Pad4): track 10.7 -> 5.55 mm
- net Net-(J8-Pad2): track 16.4 -> 13.0 mm
- net Net-(Q1-Pad2): track 9.20 -> 5.98 mm
- net Net-(J8-Pad1): track 16.4 -> 19.6 mm
- net GND: track 31.0 -> 32.7 mm
