File: reader/pcb/reader.sch (KiCad schematic (older format))
At the start: 8 parts, among them IC1 ARDUINO_PRO_MINI_5V, U1 UsbToSerial, U2 RDM6300

Commit message: Update.
Parts:
- removed IC1: ARDUINO_PRO_MINI_5V, Module:pro_mini, symbol arduino:ARDUINO_PRO_MINI_5V
- added A1: Arduino_Pro_Mini, Module:pro_mini, symbol gtrzps:Arduino_Pro_Mini
- added C1: 100u, Capacitor_THT:CP_Radial_D8.0mm_P5.00mm, symbol Device:CP
- added J1: Conn_01x04, Connector_JST:JST_PH_B4B-PH-K_1x04_P2.00mm_Vertical, symbol Connector_Generic:Conn_01x04
- BZ1: value Buzzer -> Murata PKM22EPP-40S1-B0
- R1, R2: value R -> 270
- U1: footprint (none) -> modules:UsbToSerial
Connections:
- net +5V: now also A1.21 (VCC), C1.1
- net BUZ1: now also A1.10 (D7)
- net BUZ2: now also A1.11 (D8)
- net GND: now also A1.23 (GND), A1.4 (GND), C1.2
- net GREEN: now also A1.9 (D6)
- net RED: now also A1.8 (D5)
- net TX: now also A1.6 (D3)
- net at U1.10 (GND): now also J1.4 (Pin_4)
- net at U1.7 (VCC): now also J1.1 (Pin_1)
- net at U1.8 (D+): now also J1.2 (Pin_2)
- net at U1.9 (D-): now also J1.3 (Pin_3)
- no-connect marks 2 -> 26
Other:
- moved on the sheet: U1
Changed lines of the file:
@@
 P 5800 2300
 F 0 "R1" V 5593 2300 50  0000 C CNN
-F 1 "R" V 5684 2300 50  0000 C CNN
+F 1 "270" V 5684 2300 50  0000 C CNN
 F 2 "Resistor_SMD:R_0805_2012Metric_Pad1.15x1.40mm_HandSolder" V 5730 2300 50  0001 C CNN
 F 3 "~" H 5800 2300 50  0001 C CNN
@@
 P 5800 2925
 F 0 "R2" V 5593 2925 50  0000 C CNN
-F 1 "R" V 5684 2925 50  0000 C CNN
+F 1 "270" V 5684 2925 50  0000 C CNN
 F 2 "Resistor_SMD:R_0805_2012Metric_Pad1.15x1.40mm_HandSolder" V 5730 2925 50  0001 C CNN
 F 3 "~" H 5800 2925 50  0001 C CNN
@@
 P 5725 3625
 F 0 "BZ1" H 5877 3654 50  0000 L CNN
-F 1 "Buzzer" H 5877 3563 50  0000 L CNN
+F 1 "Murata PKM22EPP-40S1-B0" H 5877 3563 50  0000 L CNN
 F 2 "modules:Buzzer_D22mm_H8mm_P10mm" V 5700 3725 50  0001 C CNN
 F 3 "~" V 5700 3725 50  0001 C CNN
@@
 Text GLabel 2500 5575 0    50   Input ~ 0
 TX
-Wire Wire Line
-	2500 5575 2725 5575
-Text GLabel 1250 3375 0    50   Input ~ 0
-RX
-Wire Wire Line
-	1250 3375 1500 3375
+Text GLabel 1225 3575 0    50   Input ~ 0
+TX
 Text GLabel 1275 3875 0    50   Input ~ 0
 GREEN
-Text GLabel 1250 3675 0    50   Input ~ 0
+Text GLabel 1250 3775 0    50   Input ~ 0
 RED
 Wire Wire Line
 	1275 3875 1500 3875
-Wire Wire Line
-	1500 3675 1250 3675
 Text GLabel 1275 3975 0    50   Input ~ 0
 BUZ1
@@
 	6650 2925 6650 2300
 $Comp
-L arduino:ARDUINO_PRO_MINI_5V IC1
-U 1 1 5EF106F6
-P 2300 3875
-F 0 "IC1" H 2275 4716 60  0000 C CNN
-F 1 "ARDUINO_PRO_MINI_5V" H 2275 4822 60  0000 C CNN
-F 2 "Module:pro_mini" H 2300 3875 50  0001 C CNN
-F 3 "" H 2300 3875 50  0001 C CNN
-	1    2300 3875
-	-1   0    0    1
-$EndComp
-$Comp
 L UsbToSerial:UsbToSerial U1
 U 1 1 5EF15F9F
-P 2300 2025
-F 0 "U1" V 2346 2403 50  0000 L CNN
-F 1 "UsbToSerial" V 2255 2403 50  0000 L CNN
-F 2 "" H 2300 2025 50  0001 C CNN
-F 3 "DOCUMENTATION" H 2300 2025 50  0001 C CNN
-	1    2300 2025
-	0    1    -1   0
-$EndComp
+P 2000 1625
+F 0 "U1" V 2046 2003 50  0000 L CNN
+F 1 "UsbToSerial" V 1955 2003 50  0000 L CNN
+F 2 "modules:UsbToSerial" H 2000 1625 50  0001 C CNN
+F 3 "DOCUMENTATION" H 2000 1625 50  0001 C CNN
+	1    2000 1625
+	1    0    0    1
+$EndComp
+Wire Wire Line
+	2725 5575 2500 5575
+NoConn ~ 1500 3275
+NoConn ~ 1500 3475
+NoConn ~ 1500 3675
+NoConn ~ 1500 4175
+NoConn ~ 1500 4275
+NoConn ~ 1500 4375
+NoConn ~ 2500 3675
+NoConn ~ 2500 3775
+NoConn ~ 2500 3875
+NoConn ~ 2500 3975
+NoConn ~ 2500 3275
+NoConn ~ 2500 3375
+$Comp
+L power:GND #PWR0101
+U 1 1 5EF66626
+P 2000 5050
+F 0 "#PWR0101" H 2000 4800 50  0001 C CNN
+F 1 "GND" H 2005 4877 50  0000 C CNN
+F 2 "" H 2000 5050 50  0001 C CNN
+F 3 "" H 2000 5050 50  0001 C CNN
+	1    2000 5050
+	1    0    0    -1
+$EndComp
+NoConn ~ 1250 1375
+NoConn ~ 1250 1475
+NoConn ~ 1250 1575
+NoConn ~ 1250 1675
+NoConn ~ 1250 1775
+NoConn ~ 1250 1875
+NoConn ~ 3525 5475
+NoConn ~ 3525 5575
+$Comp
+L gtrzps:Arduino_Pro_Mini A1
+U 1 1 5EF6AE53
+P 2000 3875
+F 0 "A1" H 2000 5056 50  0000 C CNN
+F 1 "Arduino_Pro_Mini" H 1400 4875 50  0000 C CNN
+F 2 "Module:pro_mini" H 2150 2925 50  0001 L CNN
+F 3 "" H 2000 2875 50  0001 C CNN
+	1    2000 3875
+	1    0    0    -1
+$EndComp
+Wire Wire Line
+	2000 5050 2000 4975
+Wire Wire Line
+	2100 4875 2100 4975
+Wire Wire Line
+	2100 4975 2000 4975
+Connection ~ 2000 4975
+Wire Wire Line
+	2000 4975 2000 4875
+NoConn ~ 1900 2875
+NoConn ~ 1500 4475
+NoConn ~ 1500 4575
+$Comp
+L Connector_Generic:Conn_01x04 J1
+U 1 1 5EF86283
+P 3225 1575
+F 0 "J1" H 3305 1567 50  0000 L CNN
+F 1 "Conn_01x04" H 3305 1476 50  0000 L CNN
+F 2 "Connector_JST:JST_PH_B4B-PH-K_1x04_P2.00mm_Vertical" H 3225 1575 50  0001 C CNN
+F 3 "~" H 3225 1575 50  0001 C CNN
+	1    3225 1575
+	1    0    0    -1
+$EndComp
+Wire Wire Line
+	3025 1475 2750 1475
+Wire Wire Line
+	2750 1575 3025 1575
+Wire Wire Line
+	3025 1675 2750 1675
+Wire Wire Line
+	2750 1775 3025 1775
+NoConn ~ 1500 3375
+Wire Wire Line
+	1250 3775 1500 3775
+$Comp
+L power:+5V #PWR0102
+U 1 1 5F00B0CF
+P 2100 2725
+F 0 "#PWR0102" H 2100 2575 50  0001 C CNN
+F 1 "+5V" H 2115 2898 50  0000 C CNN
+F 2 "" H 2100 2725 50  0001 C CNN
+F 3 "" H 2100 2725 50  0001 C CNN
+	1    2100 2725
+	1    0    0    -1
+$EndComp
+Wire Wire Line
+	2100 2725 2100 2875
+Wire Wire Line
+	1225 3575 1500 3575
+$Comp
+L Device:CP C1
+U 1 1 5F021B5D
+P 4450 5575
+F 0 "C1" H 4568 5621 50  0000 L CNN
+F 1 "100u" H 4568 5530 50  0000 L CNN
+F 2 "Capacitor_THT:CP_Radial_D8.0mm_P5.00mm" H 4488 5425 50  0001 C CNN
+F 3 "~" H 4450 5575 50  0001 C CNN
+	1    4450 5575
+	1    0    0    -1
+$EndComp
+Wire Wire Line
+	3175 5000 4450 5000
+Wire Wire Line
+	4450 5000 4450 5425
+Connection ~ 3175 5000
+Wire Wire Line
+	4450 5725 4450 6125
+Wire Wire Line
+	4450 6125 3175 6125
+Connection ~ 3175 6125
 $EndSCHEMATC

Commit message: Update buzzer footprint.
Parts:
- BZ1: footprint modules:Buzzer_D22mm_H8mm_P10mm -> modules:Buzzer_D22mm_H8mm_P7_10mm
Changed lines of the file:
@@
 F 0 "BZ1" H 5877 3654 50  0000 L CNN
 F 1 "Murata PKM22EPP-40S1-B0" H 5877 3563 50  0000 L CNN
-F 2 "modules:Buzzer_D22mm_H8mm_P10mm" V 5700 3725 50  0001 C CNN
+F 2 "modules:Buzzer_D22mm_H8mm_P7_10mm" V 5700 3725 50  0001 C CNN
 F 3 "~" V 5700 3725 50  0001 C CNN
 	1    5725 3625
